File: kicadtest/test022/test022.kicad_sch (KiCad schematic)
At the start: 6 parts

Commit message: add test23
Connections:
- net v1: now reaches BT1.1 (+), R1.1, RV1.1, U1.5 (V+)
- net V4: now reaches RV1.2, U1.1 (+)
- net GND: now reaches BT1.2 (-), J1.2 (Pin_2), R2.2, RV1.3, U1.3 (V-)
- net V3: now reaches R1.2, R2.1, U1.2 (-)
- net V2: now reaches J1.1 (Pin_1), U1.4
Other:
- moved on the sheet: J1
Changed lines of the file:
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@@
   (junction (at 90.17 76.2) (diameter 0) (color 0 0 0 0)
   )
+  (junction (at 91.44 76.2) (diameter 0) (color 0 0 0 0)
+  )
   (junction (at 90.17 58.42) (diameter 0) (color 0 0 0 0)
   )
+  (junction (at 118.11 58.42) (diameter 0) (color 0 0 0 0)
+  )
+  (junction (at 109.22 73.66) (diameter 0) (color 0 0 0 0)
+  )
+  (junction (at 91.44 71.12) (diameter 0) (color 0 0 0 0)
+  )
   (junction (at 97.79 58.42) (diameter 0) (color 0 0 0 0)
   )
-  (junction (at 109.22 88.9) (diameter 0) (color 0 0 0 0)
+  (junction (at 110.49 88.9) (diameter 0) (color 0 0 0 0)
   )
   (junction (at 90.17 88.9) (diameter 0) (color 0 0 0 0)
   )
+  (junction (at 118.11 88.9) (diameter 0) (color 0 0 0 0)
+  )
+  (wire (pts (xy 110.49 88.9) (xy 118.11 88.9))
+    (stroke (width 0) (type default))
+  )
   (wire (pts (xy 85.09 88.9) (xy 90.17 88.9))
     (stroke (width 0) (type default))
   )
-  (wire (pts (xy 88.9 71.12) (xy 92.71 71.12))
+  (wire (pts (xy 88.9 71.12) (xy 91.44 71.12))
     (stroke (width 0) (type default))
   )
@@
     (stroke (width 0) (type default))
   )
+  (wire (pts (xy 110.49 67.31) (xy 109.22 67.31))
+    (stroke (width 0) (type default))
+  )
   (wire (pts (xy 90.17 58.42) (xy 97.79 58.42))
     (stroke (width 0) (type default))
   )
-  (wire (pts (xy 90.17 76.2) (xy 92.71 76.2))
+  (wire (pts (xy 90.17 76.2) (xy 91.44 76.2))
+    (stroke (width 0) (type default))
+  )
+  (wire (pts (xy 99.06 86.36) (xy 91.44 86.36))
     (stroke (width 0) (type default))
   )
@@
     (stroke (width 0) (type default))
   )
+  (wire (pts (xy 91.44 76.2) (xy 92.71 76.2))
+    (stroke (width 0) (type default))
+  )
+  (wire (pts (xy 91.44 71.12) (xy 92.71 71.12))
+    (stroke (width 0) (type default))
+  )
   (wire (pts (xy 90.17 68.58) (xy 90.17 76.2))
     (stroke (width 0) (type default))
   )
+  (wire (pts (xy 109.22 73.66) (xy 110.49 73.66))
+    (stroke (width 0) (type default))
+  )
   (wire (pts (xy 118.11 58.42) (xy 118.11 63.5))
     (stroke (width 0) (type default))
@@
     (stroke (width 0) (type default))
   )
+  (wire (pts (xy 118.11 58.42) (xy 119.38 58.42))
+    (stroke (width 0) (type default))
+  )
   (wire (pts (xy 85.09 58.42) (xy 90.17 58.42))
     (stroke (width 0) (type default))
   )
-  (wire (pts (xy 97.79 88.9) (xy 109.22 88.9))
+  (wire (pts (xy 91.44 60.96) (xy 91.44 71.12))
+    (stroke (width 0) (type default))
+  )
+  (wire (pts (xy 97.79 88.9) (xy 110.49 88.9))
     (stroke (width 0) (type default))
   )
@@
     (stroke (width 0) (type default))
   )
-  (wire (pts (xy 109.22 88.9) (xy 118.11 88.9))
+  (wire (pts (xy 91.44 86.36) (xy 91.44 76.2))
     (stroke (width 0) (type default))
   )
@@
     (stroke (width 0) (type default))
   )
-  (wire (pts (xy 109.22 76.2) (xy 109.22 88.9))
+  (wire (pts (xy 110.49 76.2) (xy 110.49 88.9))
+    (stroke (width 0) (type default))
+  )
+  (wire (pts (xy 99.06 60.96) (xy 91.44 60.96))
+    (stroke (width 0) (type default))
+  )
+  (wire (pts (xy 109.22 67.31) (xy 109.22 73.66))
+    (stroke (width 0) (type default))
+  )
+  (wire (pts (xy 118.11 88.9) (xy 119.38 88.9))
     (stroke (width 0) (type default))
   )
@@
   (wire (pts (xy 85.09 74.93) (xy 85.09 88.9))
     (stroke (width 0) (type default))
+  )
+  (global_label "V4" (shape input) (at 99.06 60.96 0) (fields_autoplaced)
+    (effects (font (size 1.27 1.27)) (justify left))
+    (property "Intersheetrefs" "${INTERSHEET_REFS}" (at 104.3433 60.96 0)
+      (effects (font (size 1.27 1.27)) (justify left) hide)
+    )
+  )
+  (global_label "V3" (shape input) (at 99.06 86.36 0) (fields_autoplaced)
+    (effects (font (size 1.27 1.27)) (justify left))
+    (property "Intersheetrefs" "${INTERSHEET_REFS}" (at 104.3433 86.36 0)
+      (effects (font (size 1.27 1.27)) (justify left) hide)
+    )
+  )
+  (global_label "V2" (shape input) (at 110.49 67.31 0) (fields_autoplaced)
+    (effects (font (size 1.27 1.27)) (justify left))
+    (property "Intersheetrefs" "${INTERSHEET_REFS}" (at 115.7733 67.31 0)
+      (effects (font (size 1.27 1.27)) (justify left) hide)
+    )
+  )
+  (global_label "v1" (shape input) (at 119.38 58.42 0) (fields_autoplaced)
+    (effects (font (size 1.27 1.27)) (justify left))
+    (property "Intersheetrefs" "${INTERSHEET_REFS}" (at 124.5423 58.42 0)
+      (effects (font (size 1.27 1.27)) (justify left) hide)
+    )
+  )
+  (global_label "GND" (shape input) (at 119.38 88.9 0) (fields_autoplaced)
+    (effects (font (size 1.27 1.27)) (justify left))
+    (property "Intersheetrefs" "${INTERSHEET_REFS}" (at 126.2357 88.9 0)
+      (effects (font (size 1.27 1.27)) (justify left) hide)
+    )
   )
   (symbol (lib_id "Device:R_Potentiometer_Dual_Separate") (at 85.09 71.12 0) (unit 1)
@@
     )
   )
-  (symbol (lib_id "Connector:Screw_Terminal_01x02") (at 114.3 73.66 0) (unit 1)
+  (symbol (lib_id "Connector:Screw_Terminal_01x02") (at 115.57 73.66 0) (unit 1)
     (in_bom yes) (on_board yes) (dnp no) (fields_autoplaced)
-    (property "Reference" "J1" (at 116.84 74.93 0)
-      (effects (font (size 1.27 1.27)) (justify left))
-    )
-    (property "Value" "~" (at 116.84 76.2 0)
-      (effects (font (size 1.27 1.27)) (justify left))
-    )
-    (property "Footprint" "TerminalBlock:TerminalBlock_Altech_AK300-2_P5.00mm" (at 114.3 73.66 0)
-      (effects (font (size 1.27 1.27)) hide)
-    )
-    (property "Datasheet" "~" (at 114.3 73.66 0)
-      (effects (font (size 1.27 1.27)) hide)
-    )
+    (property "Reference" "J1" (at 118.11 74.93 0)
+      (effects (font (size 1.27 1.27)) (justify left))
+    )
+    (property "Value" "~" (at 118.11 76.2 0)
+      (effects (font (size 1.27 1.27)) (justify left))
+    )
+    (property "Footprint" "TerminalBlock:TerminalBlock_Altech_AK300-2_P5.00mm" (at 115.57 73.66 0)
+      (effects (font (size 1.27 1.27)) hide)
+    )
+    (property "Datasheet" "~" (at 115.57 73.66 0)
+      (effects (font (size 1.27 1.27)) hide)
+    )
