File: kicadtest/test022/test022.kicad_pcb (KiCad board)
At the start: 2 copper layers, 6 parts, among them J1 Screw_Terminal_01x02, U1 LM1875

Commit message: petite modif
Other:
- board outline added: 58.8 x 29 mm
Changed lines of the file:
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@@
     (fp_line (start -2.45 3.25) (end 3.5 3.25)
       (stroke (width 0.05) (type solid)) (layer "F.CrtYd"))
-    (fp_arc (start 3.5 3.25) (mid 3.809279 3.345913) (end 4.01 3.6)
+    (fp_arc (start 3.5 3.25) (mid 3.80926 3.345922) (end 4.01 3.6)
       (stroke (width 0.05) (type solid)) (layer "F.CrtYd"))
     (fp_arc (start 4.01 -3.6) (mid 3.809274 -3.345915) (end 3.5 -3.25)
@@
     )
   )
+  (gr_rect (start 97.58 69) (end 156.33 98.02)
+    (stroke (width 0.1) (type default)) (fill none) (layer "Edge.Cuts"))
   (segment (start 137.62 75.46) (end 144.94 75.46) (width 0.25) (layer "F.Cu") (net 1))
   (segment (start 144.94 75.46) (end 148.35 78.87) (width 0.25) (layer "F.Cu") (net 1))
