File: kicadtest/test021/test021.kicad_sch (KiCad schematic)
At the start: 9 parts, among them J1 Screw_Terminal_01x02, J2 Screw_Terminal_01x02, U1 LM1875

Commit message: petite modif
Parts:
- removed RV1: R_Potentiometer_Dual_Separate, symbol Device:R_Potentiometer_Dual_Separate
- removed TP1: TestPoint, Connector_Pin:Pin_D0.7mm_L6.5mm_W1.8mm_FlatFork, symbol Connector:TestPoint
- removed TP2, TP3: TestPoint, symbol Connector:TestPoint
- added RV2: 100k, Potentiometer_THT:Potentiometer_Alps_RK09L_Single_Horizontal, symbol Device:R_Potentiometer_Dual_Separate
- J1: value Screw_Terminal_01x02 -> ~
- J2: value Screw_Terminal_01x02 -> ~; footprint (none) -> TerminalBlock:TerminalBlock_Altech_AK300-2_P5.00mm
- R1: value R -> 100k; footprint (none) -> Resistor_THT:R_Axial_DIN0204_L3.6mm_D1.6mm_P5.08mm_Horizontal
- R2: value R -> 100k
- U1: value LM1875 -> ~
Connections:
- net V1: now reaches J1.1 (Pin_1), R1.1, U1.5 (V+)
- net V1: now also RV2.1
- net V3: now reaches U1.2 (-)
- net V3: now also RV2.2
- net VGND: now reaches J1.2 (Pin_2), J2.2 (Pin_2), R2.2, U1.3 (V-)
- net VGND: now also RV2.3
- net V2: now reaches R1.2, R2.1, U1.1 (+)
- net V4: now reaches J2.1 (Pin_1), U1.4
Other:
- moved on the sheet: J1, J2
