File: kicadtest/test23/test23.kicad_sch (KiCad schematic)
At the start: 6 parts

Commit message: petite modif
Parts:
- removed R1, R2, R3: 100k, Resistor_THT:R_Axial_DIN0309_L9.0mm_D3.2mm_P12.70mm_Horizontal, symbol Device:R
- BT1: value 5V -> 5
- RV1: footprint Potentiometer_THT:Potentiometer_Vishay_148E-149E_Single_Horizontal -> Potentiometer_THT:Potentiometer_Alps_RK09K_Single_Vertical
Other:
- moved on the sheet: J1
